Commit message: Arm almost ready

File: src/pos_arm/urdf/ur10_aug.xacro (robot description, xacro)
@@ -248,5 +248,5 @@
       </xacro:unless>
       <xacro:if value="${joint_limited}">
-        <limit lower="${-pi}" upper="${0}" effort="54.0" velocity="${max_velocity}"/>
+        <limit lower="${-pi}" upper="${pi}" effort="54.0" velocity="${max_velocity}"/>
       </xacro:if>
       <dynamics damping="0.0" friction="0.0"/>
